Commit message: Add files via upload

File: robot_description/urdf/robot.urdf (robot description, URDF)
Before this commit: robot my_robot, 2 links, 1 joints
Links:
- added link world
Joints:
- removed joint joint_1
- added joint base_to_first_joint: type continuous, parent base_link, child first_link, origin xyz=0 0 0.130 rpy=0 0 0
- added joint fixed: type fixed, parent world, child base_link
